File: circuits/epddriver/EPD_DRIVER.sch (EAGLE design)
At the start: 20 parts

Commit message: Fixed EPD_DRIVER schematic and created layout for it
Parts:
- removed 2N7002KW, 2N7002KW/NC: SD215, transistor-fet:SD215
- removed D1: 15KEXX, diode:15KEXX
- removed R2: 2k, SparkFun-Passives:RESISTOR0402-RES
- added !RESET, BORDER, BUSY, GND, GPIO, ICS, SCLK, SI, SO, VDD: SE11, solpad:SE11
- added B24013F: (no value), diode:SCHOTTKY-DIODESMD
- added Q1, Q2: MOSFET-NCHANNEL2N7002PW, SparkFun-DiscreteSemi:MOSFET-NCHANNEL2N7002PW
- added R1: 2K, SparkFun-Passives:RESISTOR0603-RES
Connections:
- net N$36 renamed VDL
- net N$8 renamed VCL
- removed net GND-ISO: 2N7002KW.S, 2N7002KW/NC.S, C10.1, C11.1, C12.1, C13.1, C14.1, C9.1, D1.C
- removed net N$3: PIN-3.1
- removed net N$31: PIN-32.1
- removed net N$32: PIN-33.1
- removed net N$33: C10.2, PIN-34.1
- removed net N$34: C12.2, PIN-35.1
- removed net N$35: C13.2, PIN-36.1
- removed net N$37: PIN-38.1
- removed net N$38: 2N7002KW.D
- removed net N$39: PIN-8.1
- removed net N$40: C11.2, PIN-39.1, PIN-40.1, R2.1
- removed net N$42: D1.A
- removed net N$47: C8.1
- removed net N$7: 2N7002KW/NC.D
- new net BORDER: BORDER.MP, PIN-38.1, PIN-8.1
- new net GND: B24013F.C, C10.1, C11.1, C12.1, C13.1, C14.1, C9.1, PIN-3.1, Q1.S, Q2.S
- new net N$8: GND.MP, PIN-33.1
- new net VDH: C13.2, PIN-36.1, Q1.D
- new net VGH: C10.2, PIN-34.1, Q2.D
- new net VGL: B24013F.A, C12.2, PIN-35.1
- new net VST: C11.2, PIN-39.1, PIN-40.1, R1.1
- net ICS: now also ICS.MP
- net N$1: now also SCLK.MP
- net N$2: now also BUSY.MP
- net N$24: no longer C8.2
- net N$25: now also C8.2
- net N$26: now also C8.1
- net N$29: now also R1.2; no longer R2.2
- net N$30: now also PIN-32.1, VDD.MP
- net N$4: now also SI.MP
- net N$41: now also GPIO.MP, Q1.G, Q2.G; no longer 2N7002KW.G, 2N7002KW/NC.G
- net N$5: now also SO.MP
- net N$6: now also !RESET.MP
Other:
- note removed: "Border"
- note removed: "Connect to Power Switch"
- note removed: "Connect to Timing Controller GPIO"
- note removed: "Connect to Timing Controller SPI"
- note removed: "Connect toTiming Controller SPI"
- note removed: "RESET"
- note removed: "VGH"
