File: circuits/time_circuit/time.brd (EAGLE design)
At the start: 28.9 x 38.1 mm, 8 parts, among them Y2 32.768kHz

Commit message: Update oscillator with SMT part
Parts:
- removed Y2: 32.768kHz, SparkFun-FreqCtrl:TC26H
- added Y1: (no value), SparkFun-FreqCtrl:HC49UP
- moved GND 14.4 mm to (64.8, 44.5)
Connections:
- net N$3: now also Y1.1; no longer Y2.1
- net N$4: now also Y1.2; no longer Y2.2
Changed lines of the file:
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@@
 <elements>
 <element name="DS1307" library="ds1307_pcf8583" package="DIL08" value="DS1307" x="50.8" y="48.26"/>
-<element name="GND" library="solpad" package="SE13" value="SE13" x="54.61" y="34.29"/>
+<element name="GND" library="solpad" package="SE13" value="SE13" x="64.77" y="44.45"/>
 <element name="R1" library="SparkFun-Resistors" package="0603-RES" value="10K" x="45.72" y="58.42" rot="R180">
 <attribute name="PROD_ID" value="RES-00824" x="45.72" y="58.42" size="1.778" layer="27" rot="R180" display="off"/>
@@
 <element name="SCL_RTC" library="solpad" package="SE13" value="SE13" x="52.07" y="58.42"/>
 <element name="SDA_RTC" library="solpad" package="SE13" value="SE13" x="60.96" y="63.5"/>
-<element name="Y2" library="SparkFun-FreqCtrl" package="TC26H" value="32.768kHz" x="48.26" y="40.64" rot="R180">
-<attribute name="PROD_ID" value="XTAL-10112" x="48.26" y="40.64" size="1.778" layer="27" rot="R180" display="off"/>
-</element>
 <element name="VDD" library="solpad" package="SE13" value="SE13" x="41.91" y="52.07"/>
+<element name="Y1" library="SparkFun-FreqCtrl" package="HC49UP" value="" x="49.53" y="35.56" rot="R180"/>
 </elements>
 <signals>
@@
 </signal>
 <signal name="N$3">
-<contactref element="Y2" pad="1"/>
 <contactref element="DS1307" pad="2"/>
-<wire x1="49.53" y1="44.45" x2="49.53" y2="40.64" width="0" layer="19" extent="1-1"/>
+<contactref element="Y1" pad="1"/>
+<wire x1="54.356" y1="35.56" x2="49.53" y2="44.45" width="0" layer="19" extent="1-1"/>
 </signal>
 <signal name="N$4">
 <contactref element="DS1307" pad="1"/>
-<contactref element="Y2" pad="2"/>
-<wire x1="46.99" y1="44.45" x2="46.99" y2="40.64" width="0" layer="19" extent="1-1"/>
+<contactref element="Y1" pad="2"/>
+<wire x1="44.704" y1="35.56" x2="46.99" y2="44.45" width="0" layer="19" extent="1-1"/>
 </signal>
 <signal name="GND">
@@
 <contactref element="DS1307" pad="3"/>
 <contactref element="GND" pad="MP"/>
-<wire x1="54.61" y1="44.45" x2="54.61" y2="34.29" width="0" layer="19" extent="1-1"/>
+<wire x1="54.61" y1="44.45" x2="64.77" y2="44.45" width="0" layer="19" extent="1-1"/>
 <wire x1="52.07" y1="44.45" x2="54.61" y2="44.45" width="0" layer="19" extent="1-1"/>
 </signal>
