File: circuits/MedStat/main_old.sch (EAGLE design)
At the start: 56 parts, among them U1 BLE113-VISUAL-A, U2 MMA8452Q

Commit message: branch create
Parts:
- added R12: 10k, SparkFun-Resistors:RESISTOR0603
Connections:
- new net N$49: R12.1, U1.RESET
- net VDD: now also R12.2
Changed lines of the file:
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@@
 <?xml version="1.0" encoding="utf-8"?>
 <!DOCTYPE eagle SYSTEM "eagle.dtd">
-<eagle version="7.4.0">
+<eagle version="7.2.0">
 <drawing>
 <settings>
@@
 <part name="JP1" library="SparkFun-Connectors" deviceset="USB_MICROB_PLUG" device="-SMT"/>
 <part name="GND26" library="SparkFun-Aesthetics" deviceset="GND" device=""/>
+<part name="R12" library="SparkFun-Resistors" deviceset="RESISTOR" device="0603" value="10k"/>
 </parts>
 <sheets>
@@
 <instance part="JP1" gate="G$1" x="-185.42" y="-10.16"/>
 <instance part="GND26" gate="1" x="-167.64" y="-25.4"/>
+<instance part="R12" gate="G$1" x="33.02" y="15.24" rot="R90"/>
 </instances>
 <busses>
@@
 <label x="-71.12" y="-15.24" size="1.778" layer="95"/>
 </segment>
+<segment>
+<pinref part="R12" gate="G$1" pin="2"/>
+<wire x1="33.02" y1="20.32" x2="33.02" y2="25.4" width="0.1524" layer="91"/>
+<label x="33.02" y="22.86" size="1.778" layer="95"/>
+</segment>
 </net>
 <net name="!LED_ENABLE" class="0">
@@
 </segment>
 </net>
+<net name="N$49" class="0">
+<segment>
+<pinref part="U1" gate="G$1" pin="RESET"/>
+<pinref part="R12" gate="G$1" pin="1"/>
+<wire x1="17.78" y1="5.08" x2="33.02" y2="5.08" width="0.1524" layer="91"/>
+<wire x1="33.02" y1="5.08" x2="33.02" y2="10.16" width="0.1524" layer="91"/>
+</segment>
+</net>
