File: circuits/MedStat/main.sch (EAGLE design)
At the start: 0 parts

Commit message: Completed master schematic
Parts:
- added !LED_ENABLE, !PULSE_ENABLE, B1, B2, B3, B4, B_VDD, LED_GND, LED_VDD, PROBE_I, PROBE_O, PULSE_GND, PULSE_OUT, PULSE_VDD: (no value), wirepad:SMD2
- added C1: 1uF, SparkFun-Passives:CAP0603-CAP
- added C2: 0.1uF, standardparts:CAPACITOR.0201
- added C3: 4.7uF, standardparts:CAPACITOR.0201
- added C4: 1uF, standardparts:CAPACITOR.0201
- added JP1: (no value), SparkFun-Connectors:M03X2POGO_PINS
- added R1, R5, R6, R7, R8: 10k, standardparts:RESISTOR.0201
- added R2, R3: 4.7k, standardparts:RESISTOR.0201
- added R4: 1M, standardparts:RESISTOR.0201
- added U$1: P-CHANNEL-MOSFET, GeekAmmo:P-CHANNEL-MOSFET
- added U1: BLE113-A, sf-bluegiga:BLE113-A
- added U2: MMA8452Q, SparkFun-Sensors:MMA8452Q
- added U3: BQ32000DR, Texas Instruments_By_element14_Batch_1:BQ32000DR
- added Y1: (no value), microbuilder:CRYSTAL32.768
Connections:
- new net !CHG: U$1.CHG
- new net !E_ENABLE: U$1.G
- new net !PGOOD: U$1.PGOOD
- new net !RESET: JP1.3, R1.1, U1.RESET
- new net 3.3V: B_VDD.P, C1.2, C3.1, C4.1, C4.2, JP1.1, LED_VDD.P, PULSE_VDD.P, R1.2, R2.2, R3.2, U$1.S, U1.AVDD, U1.DVDD, U2.VDD, U2.VDDIO, U3.VBACK, U3.VCC
- new net BATTERY_V+: C1.2, U$1.BAT
- new net C14M: C2.1
- new net C14P: C2.2
- new net C21M: C4.2
- new net C21P: C4.1
- new net C31M: C3.2
- new net C31P: C3.1
- new net CHG_OUT: C3.1, C4.2, U$1.OUT
- new net E_VDD: U$1.D
- new net GND: C1.1, C2.1, C3.2, C4.1, JP1.5, JP1.GND, LED_GND.P, PULSE_GND.P, R1.1, R2.1, R3.1, R4.1, R4.2, R5.1, R6.1, R7.1, R8.1, U$1.CE, U$1.EN1, U$1.EN2, U$1.TMR, U$1.VSS, U1.GND, U2.GND@0, U2.GND@1, U2.GND@2, U2.SA0, U3.GND
- new net N$1: R5.2, R6.1, U3.OSCO, Y1.2
- new net N$2: C2.2, R6.2, U2.BYP
- new net N$3: PROBE_O.P, R2.2, U$1.D, U$1.ISET
- new net N$5: R1.2, U$1.ILIM
- new net N$7: R3.2, U$1.TS
- new net OSCI: U3.OSCI, Y1.1
- new net P0_0: PULSE_OUT.P, U1.P0_0
- new net P0_1: PROBE_I.P, R4.1, U1.P0_1
- new net P0_2: U1.P0_2
- new net P0_3: U1.P0_3
- new net P0_4: U1.P0_4
- new net P0_5: U1.P0_5
- new net P0_6: U1.P0_6
- new net P0_7: U1.P0_7
- new net P1_0: U1.P1_0, U3.~IRQ
- new net P1_1: U1.P1_1
- new net P1_2: B4.P, R8.2, U1.P1_2
- new net P1_3: B3.P, R7.2, U1.P1_3
- new net P1_4: B2.P, R6.2, U1.P1_4
- new net P1_5: B1.P, R5.2, U1.P1_5
- new net P1_6: U1.P1_6
- new net P1_7: U1.P1_7
- new net P2_0: !PULSE_ENABLE.P, U1.P2_0
- new net P2_1: !LED_ENABLE.P, JP1.2, U1.P2_1
- new net P2_2: JP1.4, U$1.G, U1.P2_2
- new net SCL: R2.1, U1.SCL, U2.SCL, U3.SCL
- new net SDA: R3.1, U1.SDA, U2.SDA, U3.SDA
- new net VCC: JP1.VCC, R4.2, U$1.IN, U$1.TD
- new net VCL: C1.2
- new net VCOM_DRIVER: R1.2
- new net VST: R1.1
Other:
- note added: "ACCELEROMETER"
- note added: "BUTTONS"
- note added: "EPAPER"
- note added: "INDICATOR LEDs"
- note added: "MOISTURE"
- note added: "POWER"
- note added: "PROGRAMMER"
- note added: "PULSE"
- note added: "TIME"

Commit message: Finished final board layout round 1
Parts:
- removed B3, B4: (no value), wirepad:SMD2
- removed C4: 1uF, standardparts:CAPACITOR.0201
- removed R7, R8: 10k, standardparts:RESISTOR.0201
- C2, C3: device standardparts:CAPACITOR.0201 -> standardparts:CAPACITOR.0402
- R1, R2, R3, R4, R5, R6: device standardparts:RESISTOR.0201 -> standardparts:RESISTOR.0402
Connections:
- net C14P renamed C32M
- removed net C14M: C2.1
- removed net C21M: C4.2
- removed net C21P: C4.1
- new net C32P: C2.1
- new net VOUT: C2.1
- net 3.3V: no longer C4.1, C4.2
- net CHG_OUT: no longer C4.2
- net GND: now also C2.2; no longer C4.1, R7.1, R8.1
- net P1_2: no longer B4.P, R8.2
- net P1_3: no longer B3.P, R7.2
Other:
- moved on the sheet: B1, B2, R5, R6
